File: launch-relay.kicad_pcb (KiCad board)
At the start: 6 copper layers, 50 x 50 mm, 58 parts, among them J2 Screw_Terminal_01x03, J3 Screw_Terminal_01x03, J4 Conn_01x07_Socket, Q1 NVMFS5C460NLAFT1G-YE, Q2 NVMFS5C460NLAFT1G-YE, U1 STM32U083KCUx, U10 TPS3839DBZ, U11 SN74LVC1G74DQER, U2 MX25R3235FM1IL0, U3 BMA580, U4 ACPL-217, U5 TPS3839DBZ, U6 SN74LVC1G74DQER, U7 TPS7A2433DBVR, U8 TPS7A2433DBVR, U9 ACPL-217

Commit message: ready to review
Parts:
- removed the R12 at (179.6, 88.4)
- removed the R18 at (154.8, 77.3)
- removed the R8 at (179.6, 61.3)
- added C11: 100p, Capacitor_SMD:C_0402_1005Metric, F.Cu at (90.9, 61.8)
- added C17: 100p, Capacitor_SMD:C_0402_1005Metric, F.Cu at (103.4, 63.4)
- added G***: LOGO, HPRC_Graphics:ncsu_logo, B.Cu at (91.3, 77.3)
- added G***: LOGO, HPRC_Graphics:pcbway_logo, B.Cu at (107.4, 74.0)
- added J1: Conn_01x02_Socket, Connector_PinSocket_2.54mm:PinSocket_1x02_P2.54mm_Vertical, F.Cu at (105.2, 42.2)
- BT1, Q1, Q2: moved to B.Cu
- C1: renamed from C7; footprint Capacitor_SMD:C_0603_1608Metric -> Capacitor_SMD:C_0402_1005Metric
- C10: footprint Capacitor_SMD:C_0603_1608Metric -> Capacitor_SMD:C_0402_1005Metric
- C12: renamed from C9; footprint Capacitor_SMD:C_0603_1608Metric -> Capacitor_SMD:C_0402_1005Metric
- C13: renamed from C14; footprint Capacitor_SMD:C_0603_1608Metric -> Capacitor_SMD:C_0402_1005Metric
- C14: renamed from C17; footprint Capacitor_SMD:C_0603_1608Metric -> Capacitor_SMD:C_0402_1005Metric
- C15: renamed from C13; footprint Capacitor_SMD:C_0603_1608Metric -> Capacitor_SMD:C_0402_1005Metric
- C16: renamed from C12; footprint Capacitor_SMD:C_0603_1608Metric -> Capacitor_SMD:C_0402_1005Metric
- C18: renamed from C16; footprint Capacitor_SMD:C_0603_1608Metric -> Capacitor_SMD:C_0402_1005Metric
- C19: renamed from C15; footprint Capacitor_SMD:C_0603_1608Metric -> Capacitor_SMD:C_0402_1005Metric
- C2: renamed from C4; footprint Capacitor_SMD:C_0603_1608Metric -> Capacitor_SMD:C_0402_1005Metric
- C20: renamed from C18; footprint Capacitor_SMD:C_0603_1608Metric -> Capacitor_SMD:C_0402_1005Metric
- C3: renamed from C5; footprint Capacitor_SMD:C_0603_1608Metric -> Capacitor_SMD:C_0402_1005Metric
- C4: renamed from C6; footprint Capacitor_SMD:C_0603_1608Metric -> Capacitor_SMD:C_0402_1005Metric
- C5: renamed from C1; footprint Capacitor_SMD:C_0603_1608Metric -> Capacitor_SMD:C_0402_1005Metric
- C6: renamed from C8; footprint Capacitor_SMD:C_0603_1608Metric -> Capacitor_SMD:C_0402_1005Metric
- C7: renamed from C3; footprint Capacitor_SMD:C_0603_1608Metric -> Capacitor_SMD:C_0402_1005Metric
- C8: renamed from C2; footprint Capacitor_SMD:C_0603_1608Metric -> Capacitor_SMD:C_0402_1005Metric
- C9: renamed from C11; footprint Capacitor_SMD:C_0603_1608Metric -> Capacitor_SMD:C_0402_1005Metric
- R1: renamed from R20; footprint Resistor_SMD:R_0603_1608Metric -> Resistor_SMD:R_0402_1005Metric
- R10: renamed from R4; footprint Resistor_SMD:R_0603_1608Metric -> Resistor_SMD:R_0402_1005Metric
- R11: renamed from R5; footprint Resistor_SMD:R_0603_1608Metric -> Resistor_SMD:R_0402_1005Metric
- R12: renamed from R6; footprint Resistor_SMD:R_0603_1608Metric -> Resistor_SMD:R_0402_1005Metric
- R13: renamed from R7; footprint Resistor_SMD:R_0603_1608Metric -> Resistor_SMD:R_0402_1005Metric
- R14: renamed from R9; footprint Resistor_SMD:R_0603_1608Metric -> Resistor_SMD:R_0402_1005Metric
- R15: renamed from R13; footprint Resistor_SMD:R_0603_1608Metric -> Resistor_SMD:R_0402_1005Metric
- R16: renamed from R10; footprint Resistor_SMD:R_0603_1608Metric -> Resistor_SMD:R_0402_1005Metric
- R17: renamed from R11; value 1k -> 10k; footprint Resistor_SMD:R_0603_1608Metric -> Resistor_SMD:R_0402_1005Metric
- R18: renamed from R14; footprint Resistor_SMD:R_0603_1608Metric -> Resistor_SMD:R_0402_1005Metric
- R2: renamed from R17; footprint Resistor_SMD:R_0603_1608Metric -> Resistor_SMD:R_0402_1005Metric
- R3: renamed from R19; footprint Resistor_SMD:R_0603_1608Metric -> Resistor_SMD:R_0402_1005Metric
- R4: renamed from R21; footprint Resistor_SMD:R_0603_1608Metric -> Resistor_SMD:R_0402_1005Metric
- R5: renamed from R2; value 10k -> 4.7k; footprint Resistor_SMD:R_0603_1608Metric -> Resistor_SMD:R_0402_1005Metric
- R6: renamed from R1; value 10k -> 4.7k; footprint Resistor_SMD:R_0603_1608Metric -> Resistor_SMD:R_0402_1005Metric
- R7: renamed from R15; footprint Resistor_SMD:R_0603_1608Metric -> Resistor_SMD:R_0402_1005Metric
- R8: renamed from R16; footprint Resistor_SMD:R_0603_1608Metric -> Resistor_SMD:R_0402_1005Metric
- R9: renamed from R3; footprint Resistor_SMD:R_0603_1608Metric -> Resistor_SMD:R_0402_1005Metric
- moved U4 110.1 mm to (82.8, 61.0), turned to 90 degrees
- moved U7 109.1 mm to (92.5, 63.9)
- moved U5 106.7 mm to (88.8, 57.0), turned to -90 degrees
- moved U6 104.7 mm to (93.2, 59.6), turned to 90 degrees
- moved U11 102.9 mm to (97.5, 63.9), turned to 180 degrees
- moved U10 101.4 mm to (99.7, 59.2)
- moved J3 100.5 mm to (86.2, 68.2), turned to -90 degrees
- moved C9 97.7 mm to (82.8, 64.2)
- moved U9 97.5 mm to (103.5, 55.8), turned to -90 degrees
- moved C10 97.3 mm to (82.8, 58.0)
- moved Q1 95.5 mm to (90.9, 71.0)
- moved C12 92.3 mm to (89.0, 63.4)
- moved R15 88.9 mm to (90.8, 64.0), turned to -90 degrees
- moved C13 88.3 mm to (91.4, 58.0), turned to 180 degrees
- moved U8 88.0 mm to (108.0, 61.4), turned to 90 degrees
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- renumbered D2 to D1, D1 to D2, J4 to J2, J2 to J3, J3 to J4, U3 to U1, U1 to U2, U2 to U3, U7 to U4, U4 to U5, U5 to U6, U6 to U7
Connections:
- BT1 pad S+1: +3V0 -> Net-(J1-Pin_2)
- BT1 pad S+2: +3V0 -> Net-(J1-Pin_2)
- R14 pad 1: /Circuit Switch1/BATT_GND -> Net-(U7-C)
- R14 pad 2: Net-(U6-C) -> /Circuit Switch1/3.3V_BATT
- R17 pad 1: Net-(R11-Pad1) -> Net-(U11-C)
- R17 pad 2: Net-(U11-C) -> /Circuit Switch2/3.3V_BATT
- U2 pad 27: Net-(U1-PB4) -> /SPI3_MISO
- U5 pad 3: Net-(R8-Pad1) -> /Circuit Switch1/BATT_GND
- U5 pad 4: /Circuit Switch1/3.3V_BATT -> Net-(U7-C)
- U7 pad 1: Net-(U6-C) -> Net-(U7-C)
- U9 pad 3: Net-(R11-Pad1) -> /Circuit Switch2/BATT_GND
- U9 pad 4: /Circuit Switch2/3.3V_BATT -> Net-(U11-C)
Routing:
- net /Circuit Switch1/V_BATT: track 0.00 -> 24.3 mm
- net +3V0: track 0.00 -> 19.4 mm, vias 0 -> 14
- net Net-(Q2-G): track 0.00 -> 18.2 mm, vias 0 -> 3
- net /Flash_CS: track 0.00 -> 17.2 mm
- net /DEBUG_JTMS-SWDIO: track 0.00 -> 15.3 mm
- net /Circuit Switch2/BATT_GND: track 0.00 -> 15.1 mm, vias 0 -> 15
- net /Circuit Switch2/V_BATT: track 0.00 -> 13.2 mm
- net GND: track 0.00 -> 12.8 mm, vias 0 -> 18
- net /Circuit Switch1/BATT_GND: track 0.00 -> 11.7 mm, vias 0 -> 16
- net /BMA580_INT: track 0.00 -> 10.8 mm
- net Net-(U11-C): track 0.00 -> 10.7 mm
- net /SPI3_MISO: track 0.00 -> 10.6 mm, vias 0 -> 2
- net /DEBUG_JTCK-SWCLK: track 0.00 -> 10.3 mm
- net /Circuit Switch2/3.3V_BATT: track 0.00 -> 8.46 mm, vias 0 -> 6
- net /USART1_TX: track 0.00 -> 8.06 mm, vias 0 -> 1
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- added copper zone on B.Cu, net +3V0
- added copper zone on B.Cu, net /Circuit Switch1/3.3V_BATT
- added copper zone on B.Cu, net /Circuit Switch1/BATT_GND
- added copper zone on F.Cu, net /Circuit Switch1/BATT_GND
- added copper zone on In1.Cu, net /Circuit Switch1/BATT_GND
- added copper zone on In2.Cu, net /Circuit Switch1/BATT_GND
- added copper zone on B.Cu, net /Circuit Switch1/BATT_GND_IN
- added copper zone on F.Cu, net /Circuit Switch1/BATT_GND_IN
- added copper zone on In1.Cu, net /Circuit Switch1/BATT_GND_IN
- added copper zone on In2.Cu, net /Circuit Switch1/BATT_GND_IN
- added copper zone on B.Cu, net /Circuit Switch2/3.3V_BATT
- added copper zone on B.Cu, net /Circuit Switch2/BATT_GND
- added copper zone on F.Cu, net /Circuit Switch2/BATT_GND
- added copper zone on In1.Cu, net /Circuit Switch2/BATT_GND
- added copper zone on In2.Cu, net /Circuit Switch2/BATT_GND
- added copper zone on B.Cu, net /Circuit Switch2/BATT_GND_IN
- added copper zone on F.Cu, net /Circuit Switch2/BATT_GND_IN
- added copper zone on In1.Cu, net /Circuit Switch2/BATT_GND_IN
- added copper zone on In2.Cu, net /Circuit Switch2/BATT_GND_IN
- added copper zone on In2.Cu, net GND
- added copper zone on F.Cu, net Net-(J1-Pin_2)
- removed copper zone on In2.Cu, net +3V0
- removed copper zone on In4.Cu, net GND
Other:
- board size 50 x 50 mm -> 30 x 42 mm
- copper layers 6 -> 4
- board text added: "DUMP"
- board text added: "GND"
- board text added: "GND BATT"
- board text added: "GND LOAD"
- board text added: "LAUNCH RELAY"
- board text added: "PWR"
- board text added: "PWR IN"
- board text added: "RX"
- board text added: "SWCLK"
- board text added: "SWDIO"
- board text added: "TX"

Commit message: changes
Parts:
- removed J3, J4: Screw_Terminal_01x03, TerminalBlock_Philmore:TerminalBlock_Philmore_TB133_1x03_P5.00mm_Horizontal
- added J5: Screw_Terminal_01x03, TerminalBlock_Philmore:TerminalBlock_Philmore_TB133_1x03_P5.00mm_Horizontal, F.Cu at (86.3, 68.2)
- added J6: Screw_Terminal_01x03, TerminalBlock_Philmore:TerminalBlock_Philmore_TB133_1x03_P5.00mm_Horizontal, F.Cu at (103.8, 78.2)
- moved Q2 2.17 mm to (99.4, 73.0), turned to 0 degrees
Routing:
- net /Circuit Switch2/V_BATT: track 13.2 -> 23.8 mm
- net Net-(Q2-G): track 18.2 -> 22.1 mm, vias 3 -> 1
- net +3V0: track 19.4 -> 20.7 mm
- net /Circuit Switch2/BATT_GND_IN: vias 16 -> 14
Other:
- board text added: "BATT +"
- board text added: "BATT -"
- board text added: "LOAD GND"
- board text removed: "GND BATT"
- board text removed: "GND LOAD"
- board text removed: "PWR"
