File: launch-relay.kicad_pcb (KiCad board)
At the start: 4 copper layers, 30 x 42 mm, 64 parts, among them J1 Conn_01x02_Socket, J2 Conn_01x07_Socket, J5 Screw_Terminal_01x03, J6 Screw_Terminal_01x03, Q1 NVMFS5C460NLAFT1G-YE, Q2 NVMFS5C460NLAFT1G-YE, U1 BMA580, U10 TPS3839DBZ, U11 SN74LVC1G74DQER, U12 SN74LVC1G17DPWR, U13 SN74LVC1G17DPWR, U2 STM32U083KCUx, U3 MX25R3235FM1IL0, U4 TPS7A2450DBVR, U5 ACPL-217, U6 TPS3839DBZ, U7 SN74LVC1G74DQER, U8 TPS7A2450DBVR, U9 ACPL-217

Commit message: ordered
Parts:
- C5: value 100nF -> 100n
- moved R20 0.10 mm to (104.2, 70.2)
Other:
- outline, holes or cut-outs redrawn

Commit message: ordered fr fr
Parts:
- added H1: MountingHole, MountingHole:MountingHole_2.2mm_M2, F.Cu at (82.8, 38.0)
- added H2: MountingHole, MountingHole:MountingHole_2.2mm_M2, F.Cu at (107.0, 38.0)
- added H3: MountingHole, MountingHole:MountingHole_2.2mm_M2, F.Cu at (82.5, 83.8)
- added H4: MountingHole, MountingHole:MountingHole_2.2mm_M2, F.Cu at (107.4, 83.8)
- moved G*** 2.89 mm to (92.0, 80.2)
Other:
- board size 30 x 42 mm -> 30 x 51 mm
