File: circuit_switch.kicad_sch (KiCad schematic)
At the start: 15 parts, among them J3 Screw_Terminal_01x03, Q1 NVMFS5C460NLAFT1G-YE, U4 TPS7A2433DBVR, U5 ACPL-217, U6 TPS3839DBZ, U7 SN74LVC1G74DQER

Commit message: changes
Parts:
- removed J3: Screw_Terminal_01x03, TerminalBlock_Philmore:TerminalBlock_Philmore_TB133_1x03_P5.00mm_Horizontal, symbol Connector:Screw_Terminal_01x03
Other:
- moved on the sheet: Q1
Changed lines of the file:
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@@
-	)
-	(junction
-		(at 27.94 25.4)
-		(diameter 0)
-		(color 0 0 0 0)
 	)
 	(junction
@@
 	(wire
 		(pts
-			(xy 135.89 76.2) (xy 185.42 76.2)
+			(xy 135.89 76.2) (xy 187.96 76.2)
 		)
 		(stroke
@@
 	(wire
 		(pts
+			(xy 167.64 72.39) (xy 187.96 72.39)
+		)
+		(stroke
+			(width 0)
+			(type default)
+		)
+	)
+	(wire
+		(pts
 			(xy 128.27 43.18) (xy 128.27 30.48)
 		)
@@
 	(wire
 		(pts
-			(xy 173.99 72.39) (xy 185.42 72.39)
-		)
-		(stroke
-			(width 0)
-			(type default)
-		)
-	)
-	(wire
-		(pts
 			(xy 71.12 38.1) (xy 71.12 34.29)
 		)
@@
 	(wire
 		(pts
-			(xy 45.72 127) (xy 59.69 127)
-		)
-		(stroke
-			(width 0)
-			(type default)
-		)
-	)
-	(wire
-		(pts
 			(xy 135.89 86.36) (xy 139.7 86.36)
 		)
@@
 	(wire
 		(pts
-			(xy 45.72 129.54) (xy 59.69 129.54)
-		)
-		(stroke
-			(width 0)
-			(type default)
-		)
-	)
-	(wire
-		(pts
 			(xy 128.27 30.48) (xy 120.65 30.48)
 		)
@@
 	(wire
 		(pts
-			(xy 184.15 86.36) (xy 184.15 80.01)
-		)
-		(stroke
-			(width 0)
-			(type default)
-		)
-	)
-	(wire
-		(pts
 			(xy 87.63 93.98) (xy 87.63 92.71)
 		)
@@
 	(wire
 		(pts
-			(xy 45.72 132.08) (xy 59.69 132.08)
-		)
-		(stroke
-			(width 0)
-			(type default)
-		)
-	)
-	(wire
-		(pts
 			(xy 99.06 43.18) (xy 109.22 43.18)
 		)
@@
 	(wire
 		(pts
-			(xy 20.32 25.4) (xy 27.94 25.4)
-		)
-		(stroke
-			(width 0)
-			(type default)
-		)
-	)
-	(wire
-		(pts
-			(xy 170.18 86.36) (xy 184.15 86.36)
+			(xy 167.64 80.01) (xy 187.96 80.01)
 		)
 		(stroke
@@
 	(wire
 		(pts
-			(xy 184.15 80.01) (xy 185.42 80.01)
-		)
-		(stroke
-			(width 0)
-			(type default)
-		)
-	)
-	(wire
-		(pts
 			(xy 27.94 38.1) (xy 71.12 38.1)
 		)
@@
 			(width 0)
 			(type default)
-		)
-	)
-	(label "BATT_GND_IN"
-		(at 59.69 129.54 180)
-		(effects
-			(font
-				(size 1.27 1.27)
-			)
-			(justify right bottom)
 		)
 	)
@@
 		)
 	)
-	(label "BATT_GND"
-		(at 59.69 132.08 180)
-		(effects
-			(font
-				(size 1.27 1.27)
-			)
-			(justify right bottom)
-		)
-	)
 	(label "3.3V_BATT"
 		(at 107.95 100.33 0)
@@
 		)
 	)
+	(label "BATT_GND_IN"
+		(at 168.91 80.01 0)
+		(effects
+			(font
+				(size 1.27 1.27)
+			)
+			(justify left bottom)
+		)
+	)
 	(label "BATT_GND"
 		(at 72.39 91.44 180)
@@
 	)
 	(label "BATT_GND"
-		(at 173.99 72.39 0)
-		(effects
-			(font
-				(size 1.27 1.27)
-			)
-			(justify left bottom)
-		)
-	)
-	(label "BATT_GND"
 		(at 137.16 100.33 180)
 		(effects
@@
 		)
 	)
-	(label "BATT_GND_IN"
-		(at 170.18 86.36 0)
+	(label "BATT_GND"
+		(at 168.91 72.39 0)
 		(effects
 			(font
@@
 			)
 			(justify left bottom)
-		)
-	)
-	(label "V_BATT"
-		(at 59.69 127 180)
-		(effects
-			(font
-				(size 1.27 1.27)
-			)
-			(justify right bottom)
 		)
 	)
@@
 			)
 			(justify right bottom)
-		)
-	)
-	(label "V_BATT"
-		(at 20.32 25.4 0)
-		(effects
-			(font
-				(size 1.27 1.27)
-			)
-			(justify left bottom)
 		)
 	)
@@
 		)
 	)
-	(symbol
-		(lib_id "Connector:Screw_Terminal_01x03")
-		(at 40.64 129.54 180)
-		(unit 1)
-		(body_style 1)
-		(exclude_from_sim no)
-		(in_bom yes)
-		(on_board yes)
-		(in_pos_files yes)
-		(dnp no)
-		(fields_autoplaced yes)
-		(property "Reference" "J3"
-			(at 40.64 120.65 0)
-			(show_name no)
-			(do_not_autoplace no)
-			(effects
-				(font
-					(size 1.27 1.27)
-				)
-			)
-		)
-		(property "Value" "Screw_Terminal_01x03"
-			(at 40.64 123.19 0)
-			(show_name no)
-			(do_not_autoplace no)
-			(effects
-				(font
-					(size 1.27 1.27)
-				)
-			)
-		)
-		(property "Footprint" "TerminalBlock_Philmore:TerminalBlock_Philmore_TB133_1x03_P5.00mm_Horizontal"
-			(at 40.64 129.54 0)
-			(hide yes)
-			(show_name no)
-			(do_not_autoplace no)
-			(effects
-				(font
-					(size 1.27 1.27)
-				)
-			)
-		)
-		(property "Datasheet" ""
-			(at 40.64 129.54 0)
-			(hide yes)
-			(show_name no)
-			(do_not_autoplace no)
-			(effects
-				(font
-					(size 1.27 1.27)
-				)
-			)
-		)
-		(property "Description" "Generic screw terminal, single row, 01x03, script generated (kicad-library-utils/schlib/autogen/connector/)"
-			(at 40.64 129.54 0)
-			(hide yes)
-			(show_name no)
-			(do_not_autoplace no)
-			(effects
-				(font
-					(size 1.27 1.27)
-				)
-			)
-		)
-		(pin "3"
-		)
-		(pin "2"
-		)
-		(pin "1"
-		)
-		(instances
-			(project "launch-relay"
-				(path "/5fd10500-b703-4d79-824f-0c6e126f5ac0/addbacb5-96f0-480b-8d40-7447d1e9cbba"
-					(reference "J3")
-					(unit 1)
-				)
-				(path "/5fd10500-b703-4d79-824f-0c6e126f5ac0/fb24dfdc-7b1a-4430-ae68-8c300a39c9f8"
-					(reference "J4")
-					(unit 1)
-				)
-			)
+	(hierarchical_label "BATT_GND"
+		(shape input)
+		(at 167.64 72.39 180)
+		(effects
+			(font
+				(size 1.27 1.27)
+			)
+			(justify right)
+		)
+	)
+	(hierarchical_label "BATT_GND_IN"
+		(shape input)
+		(at 167.64 80.01 180)
+		(effects
+			(font
+				(size 1.27 1.27)
+			)
+			(justify right)
+		)
+	)
+	(hierarchical_label "V_BATT"
+		(shape input)
+		(at 27.94 25.4 180)
+		(effects
+			(font
+				(size 1.27 1.27)
+			)
+			(justify right)
 		)
 	)
@@
 	(symbol
 		(lib_id "HPRC_Logic_ICs:NVMFS5C460NLAFT1G-YE")
-		(at 185.42 71.12 0)
+		(at 187.96 71.12 0)
 		(unit 1)
 		(body_style 1)
@@
 		(fields_autoplaced yes)
 		(property "Reference" "Q1"
-			(at 207.01 74.9299 0)
+			(at 209.55 74.9299 0)
 			(show_name no)
 			(do_not_autoplace no)
@@
 		)
 		(property "Value" "NVMFS5C460NLAFT1G-YE"
-			(at 207.01 77.4699 0)
+			(at 209.55 77.4699 0)
 			(show_name no)
 			(do_not_autoplace no)
@@
 		)
 		(property "Footprint" "HPRC_Logic:NVMFS3D0P04M8LT1G"
-			(at 207.01 166.04 0)
+			(at 209.55 166.04 0)
 			(hide yes)
 			(show_name no)
@@
 		)
 		(property "Datasheet" "https://www.onsemi.com/pub/Collateral/NVMFS5C460NL-D.PDF"
-			(at 207.01 266.04 0)
+			(at 209.55 266.04 0)
 			(hide yes)
 			(show_name no)
@@
 		)
 		(property "Description" "Small Footprint (5x6 mm); Low RDS(on); RoHS Compliant; AECQ101 Qualified; Wettable Flank Option; Low QG and Capacitance"
-			(at 185.42 71.12 0)
+			(at 187.96 71.12 0)
 			(hide yes)
 			(show_name no)
@@
 		)
 		(property "Height" "1.1"
-			(at 207.01 466.04 0)
+			(at 209.55 466.04 0)
 			(hide yes)
 			(show_name no)
@@
 		)
 		(property "Manufacturer_Name" "onsemi"
-			(at 207.01 566.04 0)
+			(at 209.55 566.04 0)
 			(hide yes)
 			(show_name no)
@@
 		)
 		(property "Manufacturer_Part_Number" "NVMFS5C460NLAFT1G-YE"
-			(at 207.01 666.04 0)
+			(at 209.55 666.04 0)
 			(hide yes)
 			(show_name no)
@@
 		)
 		(property "Mouser Part Number" ""
-			(at 207.01 766.04 0)
+			(at 209.55 766.04 0)
 			(hide yes)
 			(show_name no)
@@
 		)
 		(property "Mouser Price/Stock" ""
-			(at 207.01 866.04 0)
+			(at 209.55 866.04 0)
 			(hide yes)
 			(show_name no)
@@
 		)
 		(property "Arrow Part Number" ""
-			(at 207.01 966.04 0)
+			(at 209.55 966.04 0)
 			(hide yes)
 			(show_name no)
@@
 		)
 		(property "Arrow Price/Stock" ""
-			(at 207.01 1066.04 0)
-			(hide yes)
-			(show_name no)
+			(at 209.55 1066.04 0)
+			(hide yes)
+			(show_name no)

Commit message: done
Parts:
- added R19: 100, Resistor_SMD:R_0402_1005Metric, symbol Device:R_Small
- added U12: SN74LVC1G17DPWR, HPRC_Logic:SN74LVC1G17DPWR, symbol HPRC_Logic_ICs:SN74LVC1G17DPWR
- R13: value 1k -> 330
- U4: value TPS7A2433DBVR -> TPS7A2450DBVR
Connections:
- net BATT_GND: now also U12.3 (GND)
- net at C11.2, R14.1, U5.4: now also U12.2 (A); no longer U7.1 (C)
- net at U7.5 (Q): now also R19.1; no longer Q1.4 (G)
- net 3.3V_BATT renamed 5.0V_BATT
- net 5.0V_BATT: now also U12.5 (VCC)
- new net: U12.4 (Y), U7.1 (C)
- new net: Q1.4 (G), R19.2
Other:
- moved on the sheet: C11, C12, C13, C14, Q1, R15, U6, U7

Commit message: ordered
Parts:
- C10: Manufacturer_Name (none) -> Murata Electronics; Manufacturer_Part_Number (none) -> GRT155R61A225KE01D
- C11: now left out of the parts list
- C12: Manufacturer_Name (none) -> Murata Electronics; Manufacturer_Part_Number (none) -> GRM1555C1H220JA01D
- C13, C14: Manufacturer_Name (none) -> Murata Electronics; Manufacturer_Part_Number (none) -> GRM155R61A104KA01D
- C9: Manufacturer_Name (none) -> Murata Electronics; Manufacturer_Part_Number (none) -> GRM155R61E105MA12D
- R13, R15: Manufacturer_Name (none) -> YAGEO; Manufacturer_Part_Number (none) -> RC0402FR-07330RL
- R14: Manufacturer_Name (none) -> YAGEO; Manufacturer_Part_Number (none) -> RC0402FR-0710KL
- R19: Manufacturer_Name (none) -> YAGEO; Manufacturer_Part_Number (none) -> RC0402FR-07100RL
- U12: Manufacturer_Name (none) -> Texas Instruments; Manufacturer_Part_Number (none) -> SN74LVC1G17DPWR
- U4: Manufacturer_Name (none) -> Texas Instruments; Manufacturer_Part_Number (none) -> TPS7A2450DBVR
- U5: Manufacturer_Name (none) -> Broadcom Limited; Manufacturer_Part_Number (none) -> ACPL-217-56CE
- U6: Manufacturer_Name (none) -> Texas Instruments; Manufacturer_Part_Number (none) -> TPS3839K50DBZR
- U7: Manufacturer_Name (none) -> Texas Instruments; Manufacturer_Part_Number (none) -> SN74LVC1G74DQER
