File: launch-relay.kicad_sch (KiCad schematic)
At the start: 28 parts, among them J1 Conn_01x02_Socket, J2 Conn_01x07_Socket, U1 BMA580, U2 STM32U083KCUx, U3 MX25R3235FM1IL0

Commit message: changes
Parts:
- added J5, J6: Screw_Terminal_01x03, TerminalBlock_Philmore:TerminalBlock_Philmore_TB133_1x03_P5.00mm_Horizontal, symbol Connector:Screw_Terminal_01x03
Connections:
- new net Circuit Switch1/BATT_GND: J5.1 (Pin_1)
- new net Circuit Switch1/BATT_GND_IN: J5.2 (Pin_2)
- new net Circuit Switch1/V_BATT: J5.3 (Pin_3)
- new net Circuit Switch2/BATT_GND: J6.3 (Pin_3)
- new net Circuit Switch2/BATT_GND_IN: J6.2 (Pin_2)
- new net Circuit Switch2/V_BATT: J6.1 (Pin_1)
Other:
- sheet Circuit Switch1 ports: added BATT_GND, BATT_GND_IN, V_BATT; removed none
- sheet Circuit Switch2 ports: added BATT_GND, BATT_GND_IN, V_BATT; removed none
- moved on the sheet: BT1, C6, C7, C8, J1, J2, R11, R12, U3

Commit message: ordered
Parts:
- BT1: Manufacturer_Name (none) -> MPD; Manufacturer_Part_Number (none) -> BHSD-2032-PC
- C1, C6, C7: Manufacturer_Name (none) -> Murata Electronics; Manufacturer_Part_Number (none) -> GRM155R60J475ME47D
- C2, C3, C4, C8: Manufacturer_Name (none) -> Murata Electronics; Manufacturer_Part_Number (none) -> GRM155R61A104KA01D
- C5: value 100nF -> 100n; Manufacturer_Name (none) -> Murata Electronics; Manufacturer_Part_Number (none) -> GRM155R61A104KA01D
- D1: Manufacturer_Name (none) -> Kingbright; Manufacturer_Part_Number (none) -> APT2012SURCK
- D2: Manufacturer_Name (none) -> Kingbright; Manufacturer_Part_Number (none) -> APT2012CGCK
- J1, J2, J5, J6: now left out of the parts list
- R1, R11, R12, R4: Manufacturer_Name (none) -> YAGEO; Manufacturer_Part_Number (none) -> RC0402FR-0710KL
- R10, R9: Manufacturer_Name (none) -> YAGEO; Manufacturer_Part_Number (none) -> RC0402FR-072k2L
- R2, R3, R7, R8: Manufacturer_Name (none) -> YAGEO; Manufacturer_Part_Number (none) -> RC0402FR-070RL
- R5, R6: Manufacturer_Name (none) -> YAGEO; Manufacturer_Part_Number (none) -> RC0402FR-074k7L
- U1: Manufacturer_Name (none) -> Bosch Sensortec; Manufacturer_Part_Number (none) -> BMA580
- U2: Manufacturer_Name (none) -> STMicroelectronics; Manufacturer_Part_Number (none) -> STM32U083KCU6
- U3: Manufacturer_Name (none) -> Macronix; Manufacturer_Part_Number (none) -> MX25R3235FM1IL0
