File: launch-relay.kicad_sch (KiCad schematic)
At the start: 30 parts, among them J1 Conn_01x02_Socket, J2 Conn_01x07_Socket, J5 Screw_Terminal_01x03, J6 Screw_Terminal_01x03, U1 BMA580, U2 STM32U083KCUx, U3 MX25R3235FM1IL0

Commit message: ordered fr fr
Parts:
- added H1, H2, H3, H4: MountingHole, MountingHole:MountingHole_2.2mm_M2, symbol Mechanical:MountingHole
